File: microscope_light_leds/microscope_light_leds.kicad_pcb (KiCad board)
At the start: 2 copper layers, 42.5 x 63.8 mm, 14 parts, among them J1 CONN_01x04, J2 CONN_01x04

Commit message: Finish first (and hopefully last) design of the LED ring.
Parts:
- turned LED5 to 270 degrees
Routing:
- net GND: track 0.00 -> 108.6 mm, vias 0 -> 6
- net 5v: track 0.00 -> 104.2 mm, vias 0 -> 5
- net Net-(LED5-Pad2): track 0.00 -> 12.3 mm
- net Net-(LED4-Pad2): track 0.00 -> 11.6 mm
- net Net-(LED3-Pad2): track 0.00 -> 11.5 mm
- net Net-(LED2-Pad2): track 0.00 -> 8.25 mm
- net Net-(J1-Pad2): track 0.00 -> 8.07 mm
- net Net-(J2-Pad2): track 0.00 -> 7.55 mm
- net Net-(LED1-Pad2): track 0.00 -> 6.99 mm
Other:
- board text added: "IN"
- board text added: "OUT"
