File: microscope_light_power/microscope_light_power.sch (KiCad schematic (older format))
At the start: 37 parts, among them J1 MICROUSB, J2 5V175_out, J3 enable_switch, U1 MCP73871-2AA, U2 TPS61090

Commit message: Switch the thermistor footprint to another JST PH connector. Smash everything closer together. Adjusted the test pad footprints.
Parts:
- TH1: footprint Resistors_Universal:Resistor_SMD+THTuniversal_0805to1206_RM10_HandSoldering -> Connectors_JST:JST_PH_S2B-PH-K_02x2.00mm_Angled
Changed lines of the file:
@@
 F 0 "TH1" V 4060 2550 50  0000 C CNN
 F 1 "10k" V 3890 2560 50  0000 C CNN
-F 2 "Resistors_Universal:Resistor_SMD+THTuniversal_0805to1206_RM10_HandSoldering" H 4000 2410 50  0001 C CNN
+F 2 "Connectors_JST:JST_PH_S2B-PH-K_02x2.00mm_Angled" H 4000 2410 50  0001 C CNN
 F 3 "" H 4000 2410 50  0001 C CNN
 	1    4000 2360
